File: CPU_Boards/6502_6800_CPU/6502_6800_CPU.kicad_pcb (KiCad board)
At the start: 2 copper layers, 100 x 100 mm, 91 parts, among them J1 BUS, J10 Conn_01x12, J11 Conn_01x01, J12 Conn_01x01, J13 GAL_20x10, J14 Conn_01x12, J15 Conn_01x12, J16 Conn_01x12, J17 GAL_20x10, J18 Conn_01x09, J19 Conn_01x08, J2 BUS, J20 Conn_01x08, J21 Conn_01x09, J22 JTAG, J23 Conn_01x12, J29 Conn_01x12, J3 Spare, J30 Conn_02x02_Odd_Even, J31 Conn_02x02_Odd_Even, J35 GAL_20x10, J4 Spare, J5 Conn_01x01, J6 Spare, J7 Outside, J8 Conn_01x01, J9 Conn_01x01, U2 SN74LVCC3245ANSR, U3 SN74LVC245ANSR, U4 SN74LVC245ANSR, U5 SN74LVC125AD, U6 SN74LVC125AD, U7 W65C02SxP, U9 XC9572VQ44

Commit message: first boards manufactured
Parts:
- R10, R11, R7, R8, R9: value 10k -> 1k
Changed lines of the file:
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@@
 		(sheetname "Root")
 		(sheetfile "6502_6800_CPU.kicad_sch")
-		(attr through_hole)
+		(attr through_hole exclude_from_bom)
 		(fp_line
 			(start -3.87 -1.33)
@@
 		(sheetname "Root")
 		(sheetfile "6502_6800_CPU.kicad_sch")
-		(attr through_hole)
+		(attr through_hole exclude_from_bom)
 		(fp_line
 			(start 6.46 -1.33)
@@
 		(sheetname "Root")
 		(sheetfile "6502_6800_CPU.kicad_sch")
-		(attr through_hole)
+		(attr through_hole exclude_from_bom)
 		(fp_line
 			(start 1.33 -1.33)
@@
 		(sheetfile "6502_6800_CPU.kicad_sch")
 		(zone_connect 1)
-		(attr exclude_from_pos_files)
+		(attr exclude_from_pos_files exclude_from_bom)
 		(net_tie_pad_groups "1, 2")
 		(fp_poly
@@
 		(sheetfile "6502_6800_CPU.kicad_sch")
 		(zone_connect 1)
-		(attr exclude_from_pos_files)
+		(attr exclude_from_pos_files exclude_from_bom)
 		(net_tie_pad_groups "1, 2")
 		(fp_poly
@@
 		(sheetname "Bus")
 		(sheetfile "bus.kicad_sch")
-		(attr through_hole)
+		(attr through_hole exclude_from_bom)
 		(fp_line
 			(start -3.87 49.59)
@@
 		(sheetname "Root")
 		(sheetfile "6502_6800_CPU.kicad_sch")
-		(attr through_hole)
+		(attr through_hole exclude_from_bom)
 		(fp_line
 			(start -3.87 -1.33)
@@
 		(sheetname "Root")
 		(sheetfile "6502_6800_CPU.kicad_sch")
-		(attr through_hole)
+		(attr through_hole exclude_from_bom)
 		(fp_line
 			(start 1.33 1.27)
@@
 		(sheetfile "6502_6800_CPU.kicad_sch")
 		(zone_connect 1)
-		(attr exclude_from_pos_files)
+		(attr exclude_from_pos_files exclude_from_bom)
 		(fp_line
 			(start -2.05 -1)
@@
 		(sheetname "Root")
 		(sheetfile "6502_6800_CPU.kicad_sch")
-		(attr through_hole)
+		(attr through_hole exclude_from_bom)
 		(fp_line
 			(start -1.33 -1.33)
@@
 		(sheetname "Root")
 		(sheetfile "6502_6800_CPU.kicad_sch")
-		(attr through_hole)
+		(attr through_hole exclude_from_bom)
 		(fp_line
 			(start 1.33 -1.33)
@@
 		(sheetname "Root")
 		(sheetfile "6502_6800_CPU.kicad_sch")
-		(attr through_hole)
+		(attr through_hole exclude_from_bom)
 		(fp_line
 			(start 1.33 -1.33)
@@
 		(sheetname "Root")
 		(sheetfile "6502_6800_CPU.kicad_sch")
-		(attr through_hole)
+		(attr through_hole exclude_from_bom)
 		(fp_line
 			(start 1.33 -1.33)
@@
 		(sheetname "Buffers")
 		(sheetfile "buffers.kicad_sch")
-		(attr through_hole)
+		(attr through_hole exclude_from_bom)
 		(fp_line
 			(start 1.11 0.76)
@@
 		(sheetname "Root")
 		(sheetfile "6502_6800_CPU.kicad_sch")
-		(attr through_hole)
+		(attr through_hole exclude_from_bom)
 		(fp_line
 			(start 1.33 -1.33)
@@
 		(sheetfile "buffers.kicad_sch")
 		(zone_connect 1)
-		(attr exclude_from_pos_files)
+		(attr exclude_from_pos_files exclude_from_bom)
 		(fp_line
 			(start -2.05 -1)
@@
 		(sheetfile "6502_6800_CPU.kicad_sch")
 		(zone_connect 1)
-		(attr exclude_from_pos_files)
+		(attr exclude_from_pos_files exclude_from_bom)
 		(fp_line
 			(start -2.05 -1)
@@
 		(sheetname "Root")
 		(sheetfile "6502_6800_CPU.kicad_sch")
-		(attr through_hole)
+		(attr through_hole exclude_from_bom)
 		(fp_line
 			(start -1.33 -1.33)
@@
 		(sheetfile "buffers.kicad_sch")
 		(zone_connect 1)
-		(attr exclude_from_pos_files)
+		(attr exclude_from_pos_files exclude_from_bom)
 		(fp_line
 			(start 1.4 1)
@@
 		(sheetname "Bus")
 		(sheetfile "bus.kicad_sch")
-		(attr exclude_from_pos_files)
+		(attr exclude_from_pos_files exclude_from_bom)
 		(fp_circle
 			(center 0 0)
@@
 		(sheetname "Root")
 		(sheetfile "6502_6800_CPU.kicad_sch")
-		(attr through_hole)
+		(attr through_hole exclude_from_bom)
 		(fp_line
 			(start 1.33 -0.76)
@@
 		(sheetname "Root")
 		(sheetfile "6502_6800_CPU.kicad_sch")
-		(attr through_hole)
+		(attr through_hole exclude_from_bom)
 		(fp_line
 			(start -1.33 -1.33)
@@
 		(sheetname "Buffers")
 		(sheetfile "buffers.kicad_sch")
-		(attr through_hole)
+		(attr through_hole exclude_from_bom)
 		(fp_line
 			(start -1.11 -0.76)
@@
 		(sheetfile "6502_6800_CPU.kicad_sch")
 		(zone_connect 1)
-		(attr exclude_from_pos_files)
+		(attr exclude_from_pos_files exclude_from_bom)
 		(fp_line
 			(start -2.05 0.3)
@@
 		(sheetname "Root")
 		(sheetfile "6502_6800_CPU.kicad_sch")
-		(attr through_hole)
+		(attr through_hole exclude_from_bom)
 		(fp_line
 			(start 6.46 -1.33)
@@
 		(sheetname "Root")
 		(sheetfile "6502_6800_CPU.kicad_sch")
-		(attr through_hole)
+		(attr through_hole exclude_from_bom)
 		(fp_line
 			(start 1.33 -1.33)
@@
 		(sheetfile "6502_6800_CPU.kicad_sch")
 		(zone_connect 1)
-		(attr exclude_from_pos_files)
+		(attr exclude_from_pos_files exclude_from_bom)
 		(fp_line
 			(start -2.05 0.3)
@@
 		(sheetname "Bus")
 		(sheetfile "bus.kicad_sch")
-		(attr through_hole)
+		(attr through_hole exclude_from_bom)
 		(fp_line
 			(start 1.33 -1.33)
@@
 		(sheetname "Root")
 		(sheetfile "6502_6800_CPU.kicad_sch")
-		(attr through_hole)
+		(attr through_hole exclude_from_bom)
 		(fp_line
 			(start 3.87 -1.33)
@@
 		(sheetfile "6502_6800_CPU.kicad_sch")
 		(zone_connect 1)
-		(attr exclude_from_pos_files)
+		(attr exclude_from_pos_files exclude_from_bom)
 		(net_tie_pad_groups "1, 2")
 		(fp_poly
@@
 		(sheetname "Root")
 		(sheetfile "6502_6800_CPU.kicad_sch")
-		(attr through_hole)
+		(attr through_hole exclude_from_bom)
 		(fp_line
 			(start 6.46 -1.33)
@@
 		(sheetname "Bus")
 		(sheetfile "bus.kicad_sch")
-		(attr exclude_from_pos_files)
+		(attr exclude_from_pos_files exclude_from_bom)
 		(fp_circle
 			(center 0 0)
@@
 		(sheetname "Bus")
 		(sheetfile "bus.kicad_sch")
-		(attr exclude_from_pos_files)
+		(attr exclude_from_pos_files exclude_from_bom)
 		(fp_circle
 			(center 0 0)
@@
 		(sheetname "Bus")
 		(sheetfile "bus.kicad_sch")
-		(attr exclude_from_pos_files)
+		(attr exclude_from_pos_files exclude_from_bom)
 		(fp_circle
 			(center 0 0)
@@
 		(sheetfile "6502_6800_CPU.kicad_sch")
 		(zone_connect 1)
-		(attr exclude_from_pos_files)
+		(attr exclude_from_pos_files exclude_from_bom)
 		(fp_line
 			(start -0.7 -1)
@@
 		(sheetfile "6502_6800_CPU.kicad_sch")
 		(zone_connect 1)
-		(attr exclude_from_pos_files)
+		(attr exclude_from_pos_files exclude_from_bom)
 		(fp_line
 			(start 0.7 1)
@@
 		(sheetname "Root")
 		(sheetfile "6502_6800_CPU.kicad_sch")
-		(attr through_hole)
+		(attr through_hole exclude_from_bom)
 		(fp_line
 			(start 1.06 -1)
@@
 			)
 		)
-		(property "Value" "10k"
+		(property "Value" "1k"
 			(at 0 -1.82 0)
 			(layer "B.Fab")
@@
 		(sheetfile "6502_6800_CPU.kicad_sch")
 		(zone_connect 1)
-		(attr exclude_from_pos_files)
+		(attr exclude_from_pos_files exclude_from_bom)
 		(fp_line
 			(start 1.4 -0.3)
@@
 			)
 		)
-		(property "Value" "10k"
+		(property "Value" "1k"
 			(at 0 -1.82 0)
 			(layer "B.Fab")
@@
 		(sheetfile "6502_6800_CPU.kicad_sch")
 		(zone_connect 1)
-		(attr exclude_from_pos_files)
+		(attr exclude_from_pos_files exclude_from_bom)
 		(fp_line
 			(start 1.4 -0.3)
@@
 		(sheetname "Root")
 		(sheetfile "6502_6800_CPU.kicad_sch")
-		(attr through_hole)
+		(attr through_hole exclude_from_bom)
 		(fp_line
 			(start 1.06 -1)
@@
 		(sheetfile "6502_6800_CPU.kicad_sch")
 		(zone_connect 1)
-		(attr exclude_from_pos_files)
+		(attr exclude_from_pos_files exclude_from_bom)
 		(fp_line
 			(start -0.7 -1)
@@
 		(sheetfile "6502_6800_CPU.kicad_sch")
 		(zone_connect 1)
-		(attr exclude_from_pos_files)
+		(attr exclude_from_pos_files exclude_from_bom)
 		(fp_line
 			(start 1.4 -0.3)
@@
 		(sheetfile "6502_6800_CPU.kicad_sch")
 		(zone_connect 1)
-		(attr exclude_from_pos_files)
+		(attr exclude_from_pos_files exclude_from_bom)
 		(fp_line
 			(start 1.4 -0.3)
@@
 			)
 		)
-		(property "Value" "10k"
+		(property "Value" "1k"
 			(at 0 -1.82 0)
 			(layer "B.Fab")
@@
 		(sheetfile "6502_6800_CPU.kicad_sch")
 		(zone_connect 1)
-		(attr exclude_from_pos_files)
+		(attr exclude_from_pos_files exclude_from_bom)
 		(fp_line
 			(start 0.7 1)
@@
 			)
 		)
-		(property "Value" "10k"
+		(property "Value" "1k"
 			(at 0 -1.82 0)
 			(layer "B.Fab")
@@
 		(sheetfile "6502_6800_CPU.kicad_sch")
 		(zone_connect 1)
-		(attr exclude_from_pos_files)
+		(attr exclude_from_pos_files exclude_from_bom)
 		(fp_line
 			(start 1.4 -0.3)
@@
 			)
 		)
-		(property "Value" "10k"
+		(property "Value" "1k"
 			(at 0 -1.82 0)
 			(layer "B.Fab")
@@
 		(sheetfile "6502_6800_CPU.kicad_sch")
 		(zone_connect 1)
-		(attr exclude_from_pos_files)
+		(attr exclude_from_pos_files exclude_from_bom)
 		(fp_line
 			(start 2.05 -0.3)
@@
 		(sheetfile "6502_6800_CPU.kicad_sch")
 		(zone_connect 1)
-		(attr exclude_from_pos_files)
+		(attr exclude_from_pos_files exclude_from_bom)
 		(fp_line
 			(start 1.4 -0.3)
