File: CPU_Boards/6502_6800_CPU/buffers.kicad_sch (KiCad schematic)
At the start: 16 parts, among them J11 Conn_01x01, J12 Conn_01x01, U2 SN74LVCC3245ANSR, U3 SN74LVC245ANSR, U4 SN74LVC245ANSR, U5 SN74LVC125AD, U6 SN74LVC125AD

Commit message: first boards manufactured
Parts:
- J11, J12, JP104, JP105: now left out of the parts list
Changed lines of the file:
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@@
 		(unit 1)
 		(exclude_from_sim no)
-		(in_bom yes)
+		(in_bom no)
 		(on_board yes)
 		(dnp no)
@@
 		(unit 1)
 		(exclude_from_sim no)
-		(in_bom yes)
+		(in_bom no)
 		(on_board yes)
 		(dnp no)
@@
 		(unit 1)
 		(exclude_from_sim no)
-		(in_bom yes)
+		(in_bom no)
 		(on_board yes)
 		(dnp no)
@@
 		(unit 1)
 		(exclude_from_sim no)
-		(in_bom yes)
-		(on_board yes)
-		(dnp no)
+		(in_bom no)
+		(on_board yes)
+		(dnp no)
