File: CPU_Boards/6809_CPU/6809_CPU.kicad_pcb (KiCad board)
At the start: 2 copper layers, 100 x 100 mm, 103 parts, among them J1 BUS, J10 Conn_01x01, J11 Conn_01x01, J12 Conn_01x01, J13 Conn_01x01, J14 Conn_01x01, J15 Conn_01x01, J16 ., J17 ., J18 .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

Commit message: first boards manufactured
Parts:
- R20, R21, R22, R23, R24: value 2k2 -> 1k
