File: CPU_Boards/6502_6800_CPU/schematics_v10/6502_6800_CPU.kicad_sch (KiCad schematic)
At the start: 63 parts, among them J10 Conn_01x12, J13 GAL_20x10, J14 Conn_01x12, J15 Conn_01x12, J16 Conn_01x12, J17 GAL_20x10, J18 Conn_01x09, J19 Conn_01x08, J20 Conn_01x08, J21 Conn_01x09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

Commit message: graphic updates
Parts:
- added U1: MC6800, Package_DIP:DIP-40_W15.24mm, symbol CPU_NXP_6800:MC6800
Connections:
- net +5V: now also U1.8 (VCC)
- net BE: now also U1.36 (DBE)
- net CA0: now also U1.9 (A0)
- net CA1: now also U1.10 (A1)
- net CA10: now also U1.19 (A10)
- net CA11: now also U1.20 (A11)
- net CA12: now also U1.22 (A12)
- net CA13: now also U1.23 (A13)
- net CA14: now also U1.24 (A14)
- net CA15: now also U1.25 (A15)
- net CA2: now also U1.11 (A2)
- net CA3: now also U1.12 (A3)
- net CA4: now also U1.13 (A4)
- net CA5: now also U1.14 (A5)
- net CA6: now also U1.15 (A6)
- net CA7: now also U1.16 (A7)
- net CA8: now also U1.17 (A8)
- net CA9: now also U1.18 (A9)
- net CD0: now also U1.33 (D0)
- net CD1: now also U1.32 (D1)
- net CD2: now also U1.31 (D2)
- net CD3: now also U1.30 (D3)
- net CD4: now also U1.29 (D4)
- net CD5: now also U1.28 (D5)
- net CD6: now also U1.27 (D6)
- net CD7: now also U1.26 (D7)
- net CPUCLK: no longer U8.39 (EXTAL)
- net GND: now also U1.1 (VSS), U1.21 (VSS)
- net PHI1: now also U1.3 (Phi1)
- net PHI2: now also U1.37 (Phi2)
- net RDY: now also U1.2 (~{HALT})
- net R/~{W}: now also U1.34 (R/~{W})
- net SYNC: now also U1.7 (BA)
- net ZZ39: now also U1.5 (VMA)
- net ZZ44: now also U1.40 (~{RESET})
- net ~{IRQ}: now also U1.4 (~{IRQ})
- net ~{NMI}: now also U1.6 (~{NMI})
- net Pin39: now reaches JP5.2 (C), U7.39 (ϕ2)
- net Pin39: now also U8.39 (EXTAL), U1.39 (TSC)
Other:
- note added: "6800 Signals: TSC: Three-State-Control - High active DBE: Data Bus enable - High active"
- moved on the sheet: JP3, JP4, JP5, JP6, R6, U7, U8
