File: CPU_Boards/6809_CPU/schematics_v10/6809_CPU.kicad_sch (KiCad schematic)
At the start: 68 parts, among them J16 ., J17 ., J18 ., J19 ., J20 Conn_01x12, J21 Conn_01x12, J22 Conn_01x12, J23 Conn_01x12, J24 GAL_20x10, J25 GAL_20x10, J26 Conn_01x12, J27 ., J28 ., J29 ., J32 ., J33 ., J34 JTAG, J35 Conn_01x12, J36 Spare, J37 Outside, J38 Conn_01x12, J39 GAL_20x10, J40 Conn_01x12, J41 Conn_02x02_Odd_Even, J42 Conn_02x02_Odd_Even, J5 Conn_01x09, J6 Conn_01x08, J7 Conn_01x08, J8 Conn_01x09, J9 ., U1 XC9572VQ44, U22 MC6809E, U23 MC6809

Commit message: graphic updates
Other:
- note added: "6809 Signals: Inputs on both: 3(~{IRQ}), 2(~{NMI}), 4(~{FIRQ}), 37(~{RST}), 40(~{HALT}), 39(TSC/XTAL) Outputs on both: 6(BA), 5(BS), Different signals on 6809E and 6809: 34(E - in), (E - out) 35(Q - in), (Q - out) 38(LIC - out), (EXTAL - in) 33(BUSY - out), ~{DMA/BREQ} - in) 36(AVMA - out), (MRDY - in)"
- note removed: "6809 Signals: Inputs: 3(~{IRQ}), 2(~{NMI}), 4(~{FIRQ}), 37(~{RST}), 40(~{HALT}), 39(TSC/XTAL) Outputs: 33(BUSY), 6(BA), 5(BS), 36(AVMA/MRDY) Output on 6809E (and Input on 6809): 34(E), 35(Q) 38(LIC/EXTAL) 33(BUSY/~{DMA})"
Changed lines of the file:
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@@
 		(title "Unicomp v3 - 6809 Board")
 		(date "2023-06-29")
-		(rev "v1")
+		(rev "v1.0")
 		(company "100% Offner")
 		(comment 1 "v1: Initial")
@@
 	(text "Poplate R25 and R26 for 6809.\n(~{DMA/BREQ} and MRDY)."
 		(exclude_from_sim no)
-		(at 92.71 109.855 0)
+		(at 84.074 114.3 0)
 		(effects
 			(font
@@
 		)
 	)
-	(text "6809 Signals:\nInputs:\n3(~{IRQ}), 2(~{NMI}), 4(~{FIRQ}), 37(~{RST}), 40(~{HALT}), 39(TSC/XTAL)\n\nOutputs:\n33(BUSY), 6(BA), 5(BS), 36(AVMA/MRDY)\n\nOutput on 6809E (and Input on 6809):\n34(E), 35(Q)\n38(LIC/EXTAL)\n33(BUSY/~{DMA})"
+	(text "6809 Signals:\nInputs on both:\n3(~{IRQ}), 2(~{NMI}), 4(~{FIRQ}), 37(~{RST}), 40(~{HALT}), 39(TSC/XTAL)\n\nOutputs on both:\n6(BA), 5(BS), \n\nDifferent signals \non 6809E and 6809:\n34(E - in), (E - out)\n35(Q - in), (Q - out)\n38(LIC - out), (EXTAL - in)\n33(BUSY - out), ~{DMA/BREQ} - in)\n36(AVMA - out), (MRDY - in)"
 		(exclude_from_sim no)
 		(at 185.166 51.308 0)
