File: FloppyControllerBoards/schematics_v10/WD1771_Board/WD1771_Board.kicad_sch (KiCad schematic)
At the start: 99 parts, among them J12 Floppy, J13 Test, J14 JTAG, J15 Conn_01x09, J16 Conn_01x08, J17 Conn_01x01, J18 Conn_01x01, J19 Conn_01x01, J20 Conn_01x01, J21 ~{EN}, J22 Conn_01x01, J23 Conn_01x01, J24 Conn_01x01, J25 Conn_01x01, J27 Conn_01x01, J28 Conn_01x01, J29 Conn_01x01, J30 Conn_02x02_Odd_Even, J31 Conn_02x02_Odd_Even, J32 EXT, J33 TG43, J34 READY, J35 SIDE, J6 Conn_01x09, J7 Conn_01x08, J8 E, J9 RW, U1 74HCT7540, U10 74HCT7541, U11 74HCT7540, U2 74HCT7541, U3 WD1770, U4 XC9572VQ44, U6 74ACT139, U7 WD2791, X1 8M

Commit message: graphic updates
Other:
- note added: "Adjustment Procedure: Data Separator: .) Switch on or Reset .) Ground Test Pin (TP5 - TP1) .) Observe the pulse width on pin 29 of the WD2797 (TP3) .) Adjust R4 (RPW) for 500ns Pulsewidth .) Observe the frequency on pin 16 of the WD2797 (TP4) .) Adjust C7 for 250 kHz Write Precompensation: .) Observe the pulse width on pin 31 of the WD2797 (TP2) .) Adjust R5 (WPW) for 250ns"
- note added: "For FM, DDEN# should be placed to logical "1." For MFM formats, DDEN# should be placed to a logical " 0.""
- note added: "TODO: ~{DOE} to CPLD (use DRV Pin), ~{CE1} to CPLD (with Solder Bridge), check HeadLoad end DENSEL Signal (Output or Input) and route it ot CPLD, ~{INTRQ} and DRQ to EXT Connector (J32), ch. CPLD #WG to #IDX, Make Testpoints for Adjustment (Pin16, 22, 29, 31, GND)"
Changed lines of the file:
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@@
+		)
+	)
+	(text "Adjustment Procedure:\n\nData Separator:\n.) Switch on or Reset\n.) Ground Test Pin (TP5 - TP1)\n.) Observe the pulse width on pin 29 of the WD2797 (TP3)\n.) Adjust R4 (RPW) for 500ns Pulsewidth\n.) Observe the frequency on pin 16 of the WD2797 (TP4)\n.) Adjust C7 for 250 kHz\n\nWrite Precompensation:\n.) Observe the pulse width on pin 31 of the WD2797 (TP2)\n.) Adjust R5 (WPW) for 250ns\n"
+		(exclude_from_sim no)
+		(at 217.932 198.374 0)
+		(effects
+			(font
+				(size 1.27 1.27)
+			)
+			(justify left)
 		)
 	)
@@
 		)
 	)
+	(text "TODO:\n~{DOE} to CPLD (use DRV Pin),\n~{CE1} to CPLD (with Solder Bridge),\ncheck HeadLoad end DENSEL Signal (Output or Input) and route it ot CPLD,\n~{INTRQ} and DRQ to EXT Connector (J32),\nch. CPLD #WG to #IDX,\nMake Testpoints for Adjustment (Pin16, 22, 29, 31, GND)\n\n"
+		(exclude_from_sim no)
+		(at 300.736 242.062 0)
+		(effects
+			(font
+				(size 1.27 1.27)
+			)
+			(justify left)
+		)
+	)
 	(text "Change the 7540 and 7541 to 7.5mm Package \nas they are not available in 5.3mm Package!"
 		(exclude_from_sim no)
@@
 		)
 	)
+	(text "For FM, DDEN# should be placed to logical \"1.\" \nFor MFM formats, DDEN# should be placed to a logical \" 0.\" "
+		(exclude_from_sim no)
+		(at 117.094 191.516 0)
+		(effects
+			(font
+				(size 1.27 1.27)
+			)
+			(justify left)
+		)
+	)
