File: RamRomBoard/schematics_v10/RamRomBoard.kicad_sch (KiCad schematic)
At the start: 84 parts, among them J10 Micro_SD_Card_Det2, J3 VSEL, J5 Screw_Terminal_01x02, J6 USB_B_Micro, J7 STM32F401, J8 Dual LED Socket, J9 JTAG, SW1 033TBVSA, SW2 SW_Push, U1 74LVC125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

Commit message: graphic updates
Parts:
- U12: value IS61WV10248EDBLL-10TL -> see Text
Other:
- note added: "ISSI IS61WV10248EDBLL-10TL (1MB) or Alliance AS7C34096A-10TCN (512k) or -10TIN."
- note added: "ch. CPC to ~{CNTOE} on PCB!"
Changed lines of the file:
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@@
 		)
 	)
+	(text "ch. CPC to ~{CNTOE}\non PCB!"
+		(exclude_from_sim no)
+		(at 136.652 84.074 0)
+		(effects
+			(font
+				(size 1.27 1.27)
+			)
+		)
+	)
 	(text "B10 (B11 on F103)\nB2 (B10 on F103)"
 		(exclude_from_sim no)
@@
 		)
 	)
+	(text "ISSI IS61WV10248EDBLL-10TL (1MB)\nor Alliance AS7C34096A-10TCN (512k)\nor -10TIN."
+		(exclude_from_sim no)
+		(at 274.574 235.966 0)
+		(effects
+			(font
+				(size 1.27 1.27)
+			)
+			(justify left)
+		)
+	)
 	(label "~{CERAMWR}"
 		(at 242.57 44.45 0)
@@
 			)
 		)
-		(property "Value" "IS61WV10248EDBLL-10TL"
+		(property "Value" "see Text"
 			(at 262.5441 207.01 0)
 			(effects
@@
 		(on_board yes)
 		(dnp no)
-		(fields_autoplaced yes)
 		(property "Reference" "#PWR0112"
 			(at 226.06 179.07 0)
@@
 		)
 		(property "Value" "VCCQ"
-			(at 226.06 170.18 0)
+			(at 225.806 171.196 0)
 			(effects
 				(font
